File: Inverter.kicad_sch (KiCad schematic)
At the start: 72 parts, among them Q13 CSD18540Q5B, Q14 CSD18540Q5B, Q15 CSD18540Q5B, Q16 CSD18540Q5B, Q17 CSD18540Q5B, Q18 CSD18540Q5B

Commit message: verfication inverter
Parts:
- removed C64, C76, C77, C78, C82, C83, C84, C85, C87, C88: 1u, symbol Device:C
- removed C75: 1n, symbol Device:C
- removed C86: 2.2n, symbol Device:C
- C59, C67, C74: value 1u -> 4u7 X7R 100V
- C61, C62: value 1n -> 1n X7R 100V
- C65, C66, C69: value 1u -> 100n X7R 100V
- C68: value 1u -> 1n X7R 100V
- C70: value 1u -> 2.2n
- C71, C72, C73, C79, C80, C81: value 1u -> 3n3 X7R 100V
- D10, D11, D3, D4, D5, D6, D7, D8, D9: value BAT41 -> BAT41KFILM
- R27, R28, R29: value 2.5m -> 0m5 1% 2W
- R48, R51, R53, R57, R62, R63: value 22k -> 5R 1% 0.4W
- R49, R50, R52, R54, R60, R61: value R -> 7R5 1% 1/2W
Connections:
- net +VBAT: now also C74.1; no longer C68.1, C70.1
- net GND: now also C63.2, C70.2, C74.2, D11.2 (A), D8.2 (A), NT10.2, NT12.2, R28.2, R29.2, R59.2, R65.2
- net SNC: now also C68.2
- net SPB: no longer C68.2
- net SPC: now also C68.1, C69.2
- net VSENS_C: now also C70.1
- net at C79.2, R48.1: no longer C80.2
- net at C73.2, C81.1: no longer C74.2
- net at R62.2: now also C73.1
- net at R51.1: now also C80.2; no longer C81.2
- net at R63.1: now also C81.2
- net at C71.1, R53.2: no longer C72.1
- net at C72.2, C80.1: no longer C71.2, C79.1
- new net: C72.1, R57.2
- new net: C71.2, C79.1
Other:
- note added: "1"
- note added: "2"
- note added: "3"
- note added: "4"
- note added: "Mofset : N = 6 Qg = 41 nC Qgd = 6.7 nC Rds(on),max = 2.2 mR Imax = 100 A Pcond = I*sqrt(D) Pcond,max = 9.5 W Psw = 0.5*Vbus*(tr+tf)*fpwm"
- note added: "R : protect overtensions +R better protection but slower -R faster but less protection tmiller = Qgd/Ig e.g : G current = 200mA tmiller = 33.5 ns Diodes : rapid discharge by short-circuiting the resistor"
- note added: "R shunt : current calculation I = U/R, P = R*I**2 I = 15A -> Prshunt = 0.1125W I = 30A -> Prshunt = 0.45W I = 100A -> Prshunt = 5W Vso = 1.65 + G*I*R G = (5,10,20,40) (DRV 8353) Ti recommand Vso = 0.25-3.05 V G = 20 and I = 100 -> VSO = 2.65 less R -> high current Cshunt : attnuate noise"
- note added: "RC snuber : attenuates the oscillations tau = RC = 16.5 ns fRC = 1/(2piRC) = 9.65 MHz Pr = C(Vbus**2)fpwm"
- note added: "current reserve"
- note added: "protects the MOSFET against negative voltages"
- moved on the sheet: C59, C65, D3, D4, Q14, R49, R53
