File: driver.kicad_sch (KiCad schematic)
At the start: 12 parts, among them U2 DRV8353RS

Commit message: verfication inverter
Other:
- note added: "Vcp = Vdrain +10.5V 24 + 10.5 = 34.5 Vc17 = Vcp - Vdrain 34.5 - 24 = 10.5 marge at 25V"
- note removed: "Vcp = Vdrain +10.5V 24 + 10.5 = 34.5 Vc17 = Vcp - Vdrain 34.5 - 24 = 10.5 marger à 25V"
- moved on the sheet: C19, C20
Changed lines of the file:
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@@
 	(text "7V"
 		(exclude_from_sim no)
-		(at 115.57 106.68 0)
-		(effects
-			(font
-				(size 1.27 1.27)
-			)
-		)
-	)
-	(text "Vcp = Vdrain +10.5V\n24 + 10.5 = 34.5\nVc17 = Vcp - Vdrain\n34.5 - 24 = 10.5\nmarger à 25V"
+		(at 120.65 107.95 0)
+		(effects
+			(font
+				(size 1.27 1.27)
+			)
+		)
+	)
+	(text "Vcp = Vdrain +10.5V\n24 + 10.5 = 34.5\nVc17 = Vcp - Vdrain\n34.5 - 24 = 10.5\nmarge at 25V"
 		(exclude_from_sim no)
-		(at 26.67 41.91 0)
-		(effects
-			(font
-				(size 1.27 1.27)
-			)
+		(at 17.78 44.45 0)
+		(effects
+			(font
+				(size 1.27 1.27)
+			)
+			(justify left)
 		)
 	)
@@
 	(wire
 		(pts
+			(xy 110.49 115.57) (xy 110.49 113.03)
+		)
+		(stroke
+			(width 0.3556)
+			(type default)
+			(color 0 0 0 1)
+		)
+	)
+	(wire
+		(pts
 			(xy 102.87 44.45) (xy 113.03 44.45)
 		)
@@
 	(wire
 		(pts
-			(xy 86.36 107.95) (xy 86.36 102.87)
+			(xy 86.36 105.41) (xy 86.36 102.87)
 		)
 		(stroke
@@
 	(wire
 		(pts
-			(xy 110.49 105.41) (xy 110.49 107.95)
-		)
-		(stroke
-			(width 0)
-			(type default)
-		)
-	)
-	(wire
-		(pts
 			(xy 120.65 35.56) (xy 35.56 35.56)
 		)
@@
 			(type default)
 			(color 0 0 0 1)
+		)
+	)
+	(wire
+		(pts
+			(xy 86.36 113.03) (xy 86.36 115.57)
+		)
+		(stroke
+			(width 0)
+			(type default)
 		)
 	)
@@
 	(symbol
 		(lib_id "Device:C")
-		(at 110.49 111.76 0)
+		(at 110.49 109.22 0)
 		(unit 1)
 		(body_style 1)
@@
 		(dnp no)
 		(property "Reference" "C20"
-			(at 102.87 110.49 0)
+			(at 102.87 107.95 0)
 			(show_name no)
 			(do_not_autoplace no)
@@
 		)
 		(property "Value" "470n X7R 16V"
-			(at 95.25 114.3 0)
+			(at 95.25 111.76 0)
 			(show_name no)
 			(do_not_autoplace no)
@@
 		)
 		(property "Footprint" ""
-			(at 111.4552 115.57 0)
+			(at 111.4552 113.03 0)
 			(hide yes)
 			(show_name no)
@@
 		)
 		(property "Datasheet" ""
-			(at 110.49 111.76 0)
+			(at 110.49 109.22 0)
 			(hide yes)
 			(show_name no)
@@
 		)
 		(property "Description" "Unpolarized capacitor"
-			(at 110.49 111.76 0)
+			(at 110.49 109.22 0)
 			(hide yes)
 			(show_name no)
@@
 	(symbol
 		(lib_id "Device:C")
-		(at 86.36 111.76 0)
+		(at 86.36 109.22 0)
 		(unit 1)
 		(body_style 1)
@@
 		(dnp no)
 		(property "Reference" "C19"
-			(at 80.01 109.22 0)
+			(at 80.01 106.68 0)
 			(show_name no)
 			(do_not_autoplace no)
@@
 		)
 		(property "Value" "1u X7R 25V"
-			(at 73.66 114.3 0)
+			(at 73.66 111.76 0)
 			(show_name no)
 			(do_not_autoplace no)
@@
 		)
 		(property "Footprint" ""
-			(at 87.3252 115.57 0)
+			(at 87.3252 113.03 0)
 			(hide yes)
 			(show_name no)
@@
 		)
 		(property "Datasheet" ""
-			(at 86.36 111.76 0)
+			(at 86.36 109.22 0)
 			(hide yes)
 			(show_name no)
@@
 		)
 		(property "Description" "Unpolarized capacitor"
-			(at 86.36 111.76 0)
-			(hide yes)
-			(show_name no)
+			(at 86.36 109.22 0)
+			(hide yes)
+			(show_name no)
