File: MCU.kicad_sch (KiCad schematic)
At the start: 22 parts, among them U1 STM32G474RETx, U4 PTCAN3403DRQ1, Y1 16MHz

Commit message: version before Tim
Other:
- note added: "pin 0-2 généralement utilisé pour autre chose à vérfiier"
Changed lines of the file:
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@@
+		)
+	)
+	(text "pin 0-2 généralement utilisé pour autre chose à vérfiier"
+		(exclude_from_sim no)
+		(at 226.06 48.26 0)
+		(effects
+			(font
+				(size 1.27 1.27)
+			)
 		)
 	)

Commit message: DRV et etage de puissance
Parts:
- removed C31, C32: 100n X7R 50V, symbol Device:C
- removed C33, C36: 12pf, symbol Device:C
- removed R15: 1k1, symbol Device:R
- removed R6, R7: 60 1%, symbol Device:R
- removed U4: PTCAN3403DRQ1, SOIC8_D_TEX, symbol TCAN3403DRQ1:PTCAN3403DRQ1
- removed Y1: 16MHz, symbol Device:Crystal_GND24

Commit message: verfication inverter
Other:
- moved on the sheet: C23, C24, C25, C26, C27, C29, C30, C42

Commit message: final elec V1
Parts:
- added C36: 100n X7R 10V, symbol Device:C
- added D13: SM1206NYC-IL, LED_SMD:LED_Cree-XHP50_3V_HighDensity, symbol Device:LED
- added D14: LED, LED_SMD:LED_Cree-XHP50_3V_HighDensity, symbol Device:LED
- added J6: Conn_02x05_Odd_Even, symbol Connector_Generic:Conn_02x05_Odd_Even
- added J7: Conn_01x02_Pin, Package_LCC:PLCC-84_29.3x29.3mm_P1.27mm, symbol Connector:Conn_01x02_Pin
- added Q3, Q4: PMV90ENER, 0_package_SOT_TO_SMD:SOT-23-3, symbol PMV90ENER:PMV90ENER
- added R1, R11: 100R 1% 200 mW, symbol Device:R
- added R15: 150R 1% 200 mW, symbol Device:R
- added R17: 10R 1%, symbol Device:R
- added R2: 100R 1% 200mW, symbol Device:R
- added R6, R7: 100k 1%, symbol Device:R
- added SW1: SW_Push, Button_Switch_THT:SW_NKK_GW12LJP, symbol Switch:SW_Push
Connections:
- net +3V3: now also J6.1 (Pin_1), J7.1 (Pin_1)
- net GND: now also C36.2, J6.3 (Pin_3), J6.5 (Pin_5), J6.9 (Pin_9), Q3.2 (S), Q4.2 (S), R17.2, R6.2, R7.2, SW1.1
- net LED_DBG: now also R2.1, R6.1
- net LED_PWR: now also R11.1, R7.1
- net NRST: now also C36.1, J6.10 (Pin_10), SW1.2
- net SWCLK: now also J6.4 (Pin_4)
- net SWDIO: now also J6.2 (Pin_2)
- net SENSE_TEMP_B: now reaches U1.18 (PA4)
- net SENSE_TEMP_C: now reaches U1.19 (PA5)
- net BOOT0: no longer names the net of U1.61 (PB8)
- net BOOT0: now also J7.2 (Pin_2), R17.1
- net BRAKE_PWM: no longer names the net of U1.62 (PB9)
- net CAN_INTRANET_RX: no longer names the net of U1.58 (PB5)
- net CAN_INTRANET_TX: no longer names the net of U1.59 (PB6)
- net CAN_STB: no longer names the net of U1.33 (PB11)
- net SENS_TEMP_MOFSET renamed SENSE_TEMP_A
- net SENS_TEMP_MOTOR: no longer names the net of U1.42 (PA8)
- net SENS_VBAT: no longer names the net of U1.43 (PA9)
- new net: D14.2 (A), R15.2
- new net: Q4.1 (G), R11.2
- new net: D14.1 (K), Q4.3 (D)
- new net: D13.2 (A), R1.2
- new net: Q3.1 (G), R2.2
- new net: D13.1 (K), Q3.3 (D)
- new net +5V: R1.1, R15.1
- no-connect marks 0 -> 20
Other:
- moved on the sheet: C42
