File: PCB.kicad_sch (KiCad schematic)
At the start: 0 parts

Commit message: final elec V1
Other:
- sheet MCU ports: added SENSE_TEMP_A, SENSE_TEMP_B, SENSE_TEMP_C; removed BOOT0, BRAKE_PWM, CAN_INTRANET_RX, CAN_INTRANET_TX, CAN_STB, LED_DBG, LED_PWR, NRST, SENS_TEMP_MOFSET, SENS_TEMP_MOTOR, SENS_VBAT, SWCLK, SWDIO
- sheet Sensing ports: added +A3V3, SENSE_TEMP_A, SENSE_TEMP_B, SENSE_TEMP_C; removed +A3VA, LED_DBG, LED_PWR, SENSE_TEMP_FET, SENSE_TEMP_MOT, SENSE_VBAT, VIN
