File: Sensing.kicad_sch (KiCad schematic)
At the start: 14 parts

Commit message: version before Tim
Parts:
- removed C4: 100n, symbol Device:C
- removed D13: BAT41, Diode_THT:D_DO-35_SOD27_P7.62mm_Horizontal, symbol Diode:BAT41
- removed NT2: NTC_MOT_L, Diode_THT:D_DO-35_SOD27_P7.62mm_Horizontal, symbol Device:NetTie_2
- removed R11: 2k 1%, symbol Device:R
Other:
- note removed: "Motor Temperature Sensing"

Commit message: final elec V1
Parts:
- removed D12: BAT41, Diode_THT:D_DO-35_SOD27_P7.62mm_Horizontal, symbol Diode:BAT41
- removed NT1: NTC_MOT_H, Diode_THT:D_DO-35_SOD27_P7.62mm_Horizontal, symbol Device:NetTie_2
- removed R14: 100k 1%, symbol Device:R
- removed R8: 100 1% 1/5W, symbol Device:R
- added C9: 100n X7R 10V, symbol Device:C
- added TH2, TH3: 47K 1% NTC, symbol Device:Thermistor_NTC
- C3, C5: value 100n -> 100n X7R 10V
- R12: value 4k7 1% -> 10k 1%
- R13: value 100k 1% -> 10k 1%
Connections:
- net GND: now also R13.1, C9.2
- net SENSE_TEMP_FET renamed SENSE_TEMP_A
- net SENSE_VBAT renamed SENSE_TEMP_B
- net SENSE_TEMP_B: now also TH2.2; no longer R13.1
- net VIN renamed +A3V3
- net +A3V3: now also TH2.1, TH3.1; no longer R13.2
- new net SENSE_TEMP_C: C9.1, R13.2, TH3.2
Other:
- note added: "B = 44800, Rntc = 47 000, Tntc = 298.15 K R(T) = Rntc * exp(B*(1/T - 1/Tntc) Vadc = 3.3*R/(R(T)+R) higer temp higer voltage ans lower R(T)"
- note removed: "Battery Voltage Sensing"
- note removed: "MOSFETs Temperature Sensing"
