File: motor.kicad_sch (KiCad schematic)
At the start: 29 parts, among them J1 24V, J2 5V, J3 5V, J4 USB_C_Receptacle_USB2.0_16P, J5 24V, U10 USBLC6-2SC6, U9 AM26LV32E

Commit message: version before Tim
Parts:
- C2: value C -> 0.1u X7R 10V
- R3, R4, R5: value R -> 120
Connections:
- net D+: now also R43.1; no longer R44.1
- net D-: now also R44.1; no longer R43.1
Other:
- note added: "trois test points pour les phases"
- moved on the sheet: R3, R4
Changed lines of the file:
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@@
 	(generator_version "10.0")
 	(paper "A4")
+	(text "trois test points pour les phases"
+		(exclude_from_sim no)
+		(at 160.02 100.33 0)
+		(effects
+			(font
+				(size 1.27 1.27)
+			)
+		)
+	)
 	(text "Motor phase\nMolex 39-01-2040\n"
 		(exclude_from_sim no)
@@
 	)
 	(junction
-		(at 48.26 40.64)
+		(at 45.72 40.64)
 		(diameter 0)
 		(color 0 0 0 0)
@@
 	)
 	(junction
-		(at 48.26 33.02)
+		(at 45.72 33.02)
 		(diameter 0)
 		(color 0 0 0 0)
@@
 	)
 	(junction
-		(at 49.53 50.8)
+		(at 45.72 50.8)
 		(diameter 0)
 		(color 0 0 0 0)
@@
 	)
 	(junction
-		(at 49.53 43.18)
+		(at 45.72 43.18)
 		(diameter 0)
 		(color 0 0 0 0)
@@
 		)
 	)
-	(hierarchical_label "D+"
+	(hierarchical_label "D-"
 		(shape input)
 		(at 204.47 39.37 0)
@@
 		)
 	)
-	(hierarchical_label "D-"
+	(hierarchical_label "D+"
 		(shape input)
 		(at 204.47 41.91 0)
@@
 			)
 		)
-		(property "Value" "C"
+		(property "Value" "0.1u X7R 10V"
 			(at 97.79 25.3999 0)
 			(show_name no)
@@
 	(symbol
 		(lib_id "Device:R")
-		(at 49.53 46.99 0)
+		(at 45.72 46.99 0)
 		(unit 1)
 		(body_style 1)
@@
 		(fields_autoplaced yes)
 		(property "Reference" "R4"
-			(at 52.07 45.7199 0)
+			(at 48.26 45.7199 0)
 			(show_name no)
 			(do_not_autoplace no)
@@
 			)
 		)
-		(property "Value" "R"
-			(at 52.07 48.2599 0)
+		(property "Value" "120"
+			(at 48.26 48.2599 0)
 			(show_name no)
 			(do_not_autoplace no)
@@
 		)
 		(property "Footprint" "Package_SO:SOIC-16_3.9x9.9mm_P1.27mm"
-			(at 47.752 46.99 90)
+			(at 43.942 46.99 90)
 			(hide yes)
 			(show_name no)
@@
 		)
 		(property "Datasheet" ""
-			(at 49.53 46.99 0)
+			(at 45.72 46.99 0)
 			(hide yes)
 			(show_name no)
@@
 		)
 		(property "Description" "Resistor"
-			(at 49.53 46.99 0)
+			(at 45.72 46.99 0)
 			(hide yes)
 			(show_name no)
@@
 			)
 		)
-		(property "Value" "R"
+		(property "Value" "120"
 			(at 43.18 68.5799 0)
 			(show_name no)
@@
 	(symbol
 		(lib_id "Device:R")
-		(at 48.26 36.83 0)
+		(at 45.72 36.83 0)
 		(unit 1)
 		(body_style 1)
@@
 		(fields_autoplaced yes)
 		(property "Reference" "R3"
-			(at 50.8 35.5599 0)
+			(at 48.26 35.5599 0)
 			(show_name no)
 			(do_not_autoplace no)
@@
 			)
 		)
-		(property "Value" "R"
-			(at 50.8 38.0999 0)
+		(property "Value" "120"
+			(at 48.26 38.0999 0)
 			(show_name no)
 			(do_not_autoplace no)
@@
 		)
 		(property "Footprint" "Package_SO:SOIC-16_3.9x9.9mm_P1.27mm"
-			(at 46.482 36.83 90)
+			(at 43.942 36.83 90)
 			(hide yes)
 			(show_name no)
@@
 		)
 		(property "Datasheet" ""
-			(at 48.26 36.83 0)
+			(at 45.72 36.83 0)
 			(hide yes)
 			(show_name no)
@@
 		)
 		(property "Description" "Resistor"
-			(at 48.26 36.83 0)
+			(at 45.72 36.83 0)
 			(hide yes)
 			(show_name no)

Commit message: DRV et etage de puissance
Parts:
- added C53: 1u X7R 10V, symbol Device:C
- added C58: 100n X7R 10V, symbol Device:C
- C46, C50, C51: value 470p -> 100p
- R3, R4, R5: value 120 -> 120 1%
- R38, R39, R40: value 10k -> 1k
Connections:
- net +5V: now also C53.1, C58.1
- net GND: now also C53.2, C58.2
Other:
- note added: "Hall Sensor Molex 430-45-0600 embyase mâle"
- note added: "Laisser flottant peux entrainer des commutations paraistes"
- note added: "capa : céramique C0G/NP0 10 V tol 5%"
- note added: "sortie actives si : G = 1 OU G- = 0 sorite inactive si : G = 0 ET G- = 1"
- note removed: "Hall Sensor Molex 430-25-0600"
- moved on the sheet: D1, D2, J1, J4, J5, R41, R42, R43, R44, U10

Commit message: verfication inverter
Parts:
- removed C46, C50: 100p, symbol Device:C
- removed D15, D16, D17: D, symbol Device:D
- added C57, C64: 470p COG/NP0 10V 50%, symbol Device:C
- added D18, D19, D20: PESD3V3S1UL, Diode_SMD:D_SOD-882, symbol Diode:PESD3V3S1UL
- C2: value 0.1u X7R 10V -> 100n X7R 10V
- C51: value 100p -> 470p COG/NP0 10V 50%
- R35, R36, R37: value 4.7k -> 4.7k 1%
Connections:
- net GND: now also C57.2, C64.2, D18.2 (A), D19.2 (A), D20.2 (A)
- net Hall_A: now also C64.1
- net Hall_B: now also C57.1
- net at J2.1 (Pin_1), R35.2, R38.1: now also D20.1 (K)
- net at J2.3 (Pin_3), R37.2, R40.1: now also D18.1 (K)
- net at J2.2 (Pin_2), R36.2, R39.1: now also D19.1 (K)
Other:
- note added: "Hall Sensor Molex 430-45-0600 embase mâle"
- note added: "Pr = Vdiff**2/RT"
- note added: "filtre passe-bas pour atténuer PWM : tau = RC tau,montee = (Rpull-up + Rserie)*C t10-90 = 2.2tau taudescente = Rserie*C Rserie = 1k C = 470 pF tmontee = 1.25 us tdescent = 0.22us"
- note added: "output of Hall Sensor is an open collector"
- note added: "pull-up resitance Ipull-up = 3.3/Rpull-up = 0.702 mA P = U*I = 2.32 mW"
- note removed: "Hall Sensor Molex 430-45-0600 embyase mâle"
- note removed: "capa : céramique C0G/NP0 10 V tol 5%"
- moved on the sheet: C51

Commit message: final elec V1
Parts:
- removed D18, D19, D20: PESD3V3S1UL, Diode_SMD:D_SOD-882, symbol Diode:PESD3V3S1UL
- added CR1, CR2, CR3: ESD321DYAR, SOT5x3_DYA_TEX, symbol ESD321DYAR:ESD321DYAR
- added D15: LED, LED_SMD:LED_Cree-XHP50_3V_HighDensity, symbol Device:LED
- added R45: 15k 1% 250 mW, symbol Device:R
- R43, R44: value 5k1 -> 0R
Connections:
- net +VBAT: now also R45.2
- net GND: now also CR1.1 (GND), CR2.1 (GND), CR3.1 (GND)
- net GNDPWR: now also D15.1 (K)
- net at J2.1 (Pin_1), R35.2, R38.1: now also CR3.2 (I/O)
- net at J2.3 (Pin_3), R37.2, R40.1: now also CR1.2 (I/O)
- net at J2.2 (Pin_2), R36.2, R39.1: now also CR2.2 (I/O)
- net +5V_USB_C: now reaches J4.A4 (VBUS), J4.A9 (VBUS), J4.B4 (VBUS), J4.B9 (VBUS)
- new net: D15.2 (A), R45.1
- no-connect marks 8 -> 7
Other:
- moved on the sheet: D1, D2, J5
